Commit message: Fix mesh URLs after wato_rover -> wato_uwrt_rover rename

File: src/gazebo/launch/mars_env.urdf (robot description, URDF)
Before this commit: robot mars_environment, 5 links, 4 joints
Links:
- link desert: geometry collision mesh filename=https://raw.githubusercontent.com/WATonomous/wato_uwrt_rove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 scale=0.1 0.1 0.1; visual mesh filename=https://raw.githubusercontent.com/WATonomous/wato_uwrt_rove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 scale=0.1 0.1 0.1
- link mallet: geometry collision mesh filename=https://raw.githubusercontent.com/WATonomous/wato_uwrt_rove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 scale=0.4 0.4 0.4; visual mesh filename=https://raw.githubusercontent.com/WATonomous/wato_uwrt_rove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 scale=0.4 0.4 0.4
- link water_bottle: geometry collision mesh filename=https://raw.githubusercontent.com/WATonomous/wato_uwrt_rove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 scale=0.4 0.4 0.4; visual mesh filename=https://raw.githubusercontent.com/WATonomous/wato_uwrt_rove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 scale=0.4 0.4 0.4

File: src/gazebo/launch/robot.urdf (robot description, URDF)
Before this commit: robot robot, 7 links, 6 joints
Links:
- link robot/chassis: geometry visual mesh filename=https://raw.githubusercontent.com/WATonomous/wato_uwrt_rove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
- link robot/fl_whl: geometry visual mesh filename=https://raw.githubusercontent.com/WATonomous/wato_uwrt_rove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
- link robot/fr_whl: geometry visual mesh filename=https://raw.githubusercontent.com/WATonomous/wato_uwrt_rove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
- link robot/left_wheel: geometry visual mesh filename=https://raw.githubusercontent.com/WATonomous/wato_uwrt_rove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
- link robot/right_wheel: geometry visual mesh filename=https://raw.githubusercontent.com/WATonomous/wato_uwrt_rove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
- link robot/rl_whl: geometry visual mesh filename=https://raw.githubusercontent.com/WATonomous/wato_uwrt_rove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
- link robot/rr_whl: geometry visual mesh filename=https://raw.githubusercontent.com/WATonomous/wato_uwrt_rove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

Commit message: fixed to relative paths for stl files

File: src/gazebo/launch/mars_env.urdf (robot description, URDF)
Before this commit: robot mars_environment, 5 links, 4 joints
Links:
- link desert: geometry collision mesh filename=./mars.stl scale=0.1 0.1 0.1; visual mesh filename=./mars.stl scale=0.1 0.1 0.1
- link mallet: geometry collision mesh filename=./mallet.stl scale=0.4 0.4 0.4; visual mesh filename=./mallet.stl scale=0.4 0.4 0.4
- link water_bottle: geometry collision mesh filename=./water_bottle.stl scale=0.4 0.4 0.4; visual mesh filename=./water_bottle.stl scale=0.4 0.4 0.4

File: src/gazebo/launch/robot.urdf (robot description, URDF)
Before this commit: robot robot, 7 links, 6 joints
Links:
- link robot/chassis: geometry visual mesh filename=./rover_base_link.stl
- link robot/fl_whl: geometry visual mesh filename=./rover_front_left_wheel.stl
- link robot/fr_whl: geometry visual mesh filename=./rover_front_right_wheel.stl
- link robot/left_wheel: geometry visual mesh filename=./rover_center_left_wheel.stl
- link robot/right_wheel: geometry visual mesh filename=./rover_center_right_wheel.stl
- link robot/rl_whl: geometry visual mesh filename=./rover_rear_left_wheel.stl
- link robot/rr_whl: geometry visual mesh filename=./rover_rear_right_wheel.stl
